File: kicad/Securityfest_2019_badge_beta.kicad_pcb (KiCad board)
At the start: 2 copper layers, 76.2 x 82.8 mm, 43 parts, among them J1 Micro_USB, J2 JST_CHARGE, SW1 A, SW2 B, SW3 RESET, U1 MCP73831T-2ACI_OT, U2 LD1117V33, U3 Nokia_5110_LCD, U4 ESP-12S

Commit message: Wtf?
Parts:
- moved TX/RX 24.3 mm to (139.2, 56.6), turned to 19 degrees
Routing:
- net Net-(J4-Pad2): track 3.54 -> 39.7 mm
- net Net-(J4-Pad1): track 3.64 -> 38.9 mm
- net GND: track 309.0 -> 301.7 mm
