File: kicad/Securityfest_2019_badge_beta.sch (KiCad schematic (older format))
At the start: 41 parts, among them J1 Micro_USB, J2 JST_CHARGE, J3 GPIO16, J4 TX/RX, SW1 A, SW2 B, SW3 RESET, U1 MCP73831T-2ACI_OT, U2 LD1117V33, U3 Nokia_5110_LCD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

Commit message: Wtf?
Parts:
- R14: value 10k -> 1k
Changed lines of the file:
@@
 Title "Security fest 2019 Badge"
 Date "2018-12-05"
-Rev "1.0"
+Rev "2.0"
 Comp "Security fest"
 Comment1 ""
@@
 P 9750 5100
 F 0 "R14" V 9750 5000 50  0001 L CNN
-F 1 "10k" V 9750 5050 50  0000 L CNN
+F 1 "1k" V 9750 5050 50  0000 L CNN
 F 2 "Resistors_SMD:R_0603_HandSoldering" V 9680 5100 50  0001 C CNN
 F 3 "~" H 9750 5100 50  0001 C CNN
